File: main.kicad_pcb (KiCad board)
At the start: 2 copper layers, 0 parts

Commit message: made PCB and updated Jornal
Parts:
- added A1: RaspberryPi_Pico, Module:RaspberryPi_Pico_Common_Unspecified, F.Cu at (189.0, 84.5)
- added D1: 1N4148, Diode_THT:D_DO-35_SOD27_P7.62mm_Horizontal, F.Cu at (130.5, 67.3)
- added D2: 1N4148, Diode_THT:D_DO-35_SOD27_P7.62mm_Horizontal, F.Cu at (130.5, 86.6)
- added D3: 1N4148, Diode_THT:D_DO-35_SOD27_P7.62mm_Horizontal, F.Cu at (130.5, 105.6)
- added D4: 1N4148, Diode_THT:D_DO-35_SOD27_P7.62mm_Horizontal, F.Cu at (149.5, 67.3)
- added D5: 1N4148, Diode_THT:D_DO-35_SOD27_P7.62mm_Horizontal, F.Cu at (149.5, 86.6)
- added D6: 1N4148, Diode_THT:D_DO-35_SOD27_P7.62mm_Horizontal, F.Cu at (149.5, 105.6)
- added D7: 1N4148, Diode_THT:D_DO-35_SOD27_P7.62mm_Horizontal, F.Cu at (168.5, 67.1)
- added D8: 1N4148, Diode_THT:D_DO-35_SOD27_P7.62mm_Horizontal, F.Cu at (168.5, 86.6)
- added D9: 1N4148, Diode_THT:D_DO-35_SOD27_P7.62mm_Horizontal, F.Cu at (168.5, 105.6)
- added SW1: Switch, ScottoKeebs_MX:MX_PCB_1.00u, F.Cu at (122.0, 65.0)
- added SW2: Switch, ScottoKeebs_MX:MX_PCB_1.00u, F.Cu at (121.9, 84.0)
- added SW3: Switch, ScottoKeebs_MX:MX_PCB_1.00u, F.Cu at (121.9, 103.0)
- added SW4: Switch, ScottoKeebs_MX:MX_PCB_1.00u, F.Cu at (140.9, 65.0)
- added SW5: Switch, ScottoKeebs_MX:MX_PCB_1.00u, F.Cu at (140.9, 84.0)
- added SW6: Switch, ScottoKeebs_MX:MX_PCB_1.00u, F.Cu at (140.9, 103.0)
- added SW7: Switch, ScottoKeebs_MX:MX_PCB_1.00u, F.Cu at (160.0, 64.9)
- added SW8: Switch, ScottoKeebs_MX:MX_PCB_1.00u, F.Cu at (159.9, 84.0)
- added SW9: Switch, ScottoKeebs_MX:MX_PCB_1.00u, F.Cu at (159.9, 103.0)
Routing:
- net row 2: track 0.00 -> 142.4 mm
- net col 3: track 0.00 -> 113.5 mm
- net row 3: track 0.00 -> 104.3 mm
- net Net-(A1-GPIO0): track 0.00 -> 104.0 mm
- net col2: track 0.00 -> 56.3 mm
- net col 1: track 0.00 -> 54.9 mm
- net Net-(D4-A): track 0.00 -> 6.14 mm
- net Net-(D7-A): track 0.00 -> 6.13 mm
- net Net-(D3-A): track 0.00 -> 6.07 mm
- net Net-(D2-A): track 0.00 -> 6.07 mm
- net Net-(D9-A): track 0.00 -> 6.07 mm
- net Net-(D8-A): track 0.00 -> 6.07 mm
- net Net-(D6-A): track 0.00 -> 6.07 mm
- net Net-(D5-A): track 0.00 -> 6.07 mm
- net Net-(D1-A): track 0.00 -> 6.06 mm
- added copper zone on B.Cu, net (none)
- added copper zone on F.Cu, net (none)
